File: Kicad/Stereo/troubleSeeker.kicad_pcb (KiCad board)
At the start: 2 copper layers, 35.6 x 142.9 mm, 19 parts, among them J1 Screw_Terminal_01x02, J2 AudioJack2, SW1 SW_DPST_x2, U1 TL072

Commit message: Replaced switch
Parts:
- added JP1: Jumper_2_Open, Jumper:SolderJumper-2_P1.3mm_Open_RoundedPad1.0x1.5mm, F.Cu at (158.0, 65.7)
- added JP2: Jumper_2_Open, Jumper:SolderJumper-2_P1.3mm_Open_RoundedPad1.0x1.5mm, B.Cu at (129.0, 66.2)
- added JP3: Jumper_2_Open, Jumper:SolderJumper-2_P1.3mm_Open_RoundedPad1.0x1.5mm, F.Cu at (158.0, 165.3)
- added JP4: Jumper_2_Open, Jumper:SolderJumper-2_P1.3mm_Open_RoundedPad1.0x1.5mm, B.Cu at (128.5, 165.3)
- SW1: value SW_DPST_x2 -> SW_SPDT; footprint Button_Switch_THT:SW_Push_2P1T_Toggle_CK_PVA1xxH1xxxxxxV2 -> Button_Switch_THT:SW_Slide_SPDT_Angled_CK_OS102011MA1Q
- moved SW1 9.17 mm to (131.0, 99.5), turned to -90 degrees
Connections:
- SW1 pad 1: 4.5V -> unconnected-(SW1-A-Pad1)
- SW1 pad 3: (no net) -> 4.5V
Routing:
- net Net-(JP2-A): track 0.00 -> 98.4 mm
- net Net-(JP1-B): track 0.00 -> 98.4 mm
- net Net-(J1-Pin_1): track 30.9 -> 41.6 mm
- net 4.5V: track 125.8 -> 120.9 mm
- net VGND2: track 217.1 -> 214.2 mm
- net Net-(BT1-+): track 16.2 -> 13.4 mm
- net AUDIO_R: track 129.4 -> 126.7 mm
- net Net-(J1-Pin_2): track 44.7 -> 46.8 mm
- net -4.5V: track 141.3 -> 139.5 mm
- net AUDIO_L: track 141.2 -> 139.9 mm
